Commit message: minitaur_animation

File: frost-dev-master/example/minitaur/urdf/minitaur2.urdf (robot description, URDF)
Before this commit: robot minitaur, 17 links, 16 joints
Joints:
- joint knee_back_leftL_link: limit lower=0 upper=+1.57 effort=100 velocity=1000 -> lower=0 upper=+3.1416 effort=100 velocity=1000
- joint knee_back_leftR_link: limit lower=0 upper=+1.57 effort=100 velocity=1000 -> lower=0 upper=+3.1416 effort=100 velocity=1000
- joint knee_back_rightL_link: limit lower=0 upper=+1.57 effort=100 velocity=1000 -> lower=0 upper=+3.1416 effort=100 velocity=1000
- joint knee_back_rightR_link: limit lower=0 upper=+1.57 effort=100 velocity=1000 -> lower=0 upper=+3.1416 effort=100 velocity=1000
- joint knee_front_leftL_link: limit lower=0 upper=+1.57 effort=100 velocity=1000 -> lower=0 upper=+3.1416 effort=100 velocity=1000
- joint knee_front_leftR_link: limit lower=0 upper=+1.57 effort=100 velocity=1000 -> lower=0 upper=+3.1416 effort=100 velocity=1000
- joint knee_front_rightL_link: limit lower=0 upper=+1.57 effort=100 velocity=1000 -> lower=0 upper=+3.1416 effort=100 velocity=1000
- joint knee_front_rightR_link: limit lower=0 upper=1.57 effort=100 velocity=1000 -> lower=0 upper=3.1416 effort=100 velocity=1000
- joint motor_back_leftL_joint: limit lower=-0.7854 upper=+0.7854 effort=100 velocity=1000 -> lower=0 upper=+4.7124 effort=100 velocity=1000
- joint motor_back_leftR_joint: limit lower=0.7854 upper=+2.3562 effort=100 velocity=1000 -> lower=0 upper=+4.7124 effort=100 velocity=1000
- joint motor_back_rightL_joint: limit lower=0.7854 upper=+2.3562 effort=100 velocity=1000 -> lower=0 upper=+4.7124 effort=100 velocity=1000
- joint motor_back_rightR_joint: limit lower=-0.7854 upper=+0.7854 effort=100 velocity=1000 -> lower=0 upper=+4.7124 effort=100 velocity=1000
- joint motor_front_leftL_joint: limit lower=-0.7854 upper=+0.7854 effort=100 velocity=1000 -> lower=0 upper=+4.7124 effort=100 velocity=1000
- joint motor_front_leftR_joint: limit lower=+0.7854 upper=+2.3562 effort=100 velocity=1000 -> lower=0 upper=+4.7124 effort=100 velocity=1000
- joint motor_front_rightL_joint: limit lower=0.7854 upper=+2.3562 effort=100 velocity=1000 -> lower=0 upper=+4.7124 effort=100 velocity=1000
- joint motor_front_rightR_joint: limit lower=-0.7854 upper=+0.7854 effort=100 velocity=1000 -> lower=0 upper=+4.7124 effort=100 velocity=1000

Commit message: minitaur_test_1

File: frost-dev-master/example/minitaur/urdf/minitaur2.urdf (robot description, URDF)
Before this commit: robot minitaur, 17 links, 16 joints
Joints:
- joint knee_back_leftL_link: limit lower=0 upper=+3.1416 effort=100 velocity=1000 -> lower=+0.5236 upper=+1.5708 effort=100 velocity=20
- joint knee_back_leftR_link: limit lower=0 upper=+3.1416 effort=100 velocity=1000 -> lower=+0.5236 upper=+1.5708 effort=100 velocity=20
- joint knee_back_rightL_link: limit lower=0 upper=+3.1416 effort=100 velocity=1000 -> lower=+0.5236 upper=+1.5708 effort=100 velocity=20
- joint knee_back_rightR_link: limit lower=0 upper=+3.1416 effort=100 velocity=1000 -> lower=+0.5236 upper=+1.5708 effort=100 velocity=20
- joint knee_front_leftL_link: limit lower=0 upper=+3.1416 effort=100 velocity=1000 -> lower=+0.5236 upper=+1.5708 effort=100 velocity=20
- joint knee_front_leftR_link: limit lower=0 upper=+3.1416 effort=100 velocity=1000 -> lower=+0.5236 upper=+1.5708 effort=100 velocity=20
- joint knee_front_rightL_link: limit lower=0 upper=+3.1416 effort=100 velocity=1000 -> lower=+0.5236 upper=+1.5708 effort=100 velocity=20
- joint knee_front_rightR_link: limit lower=0 upper=3.1416 effort=100 velocity=1000 -> lower=+0.5236 upper=+1.5708 effort=100 velocity=20
- joint motor_back_leftL_joint: limit lower=0 upper=+4.7124 effort=100 velocity=1000 -> lower=0 upper=+3.1416 effort=100 velocity=20
- joint motor_back_leftR_joint: limit lower=0 upper=+4.7124 effort=100 velocity=1000 -> lower=0 upper=+3.1416 effort=100 velocity=20
- joint motor_back_rightL_joint: limit lower=0 upper=+4.7124 effort=100 velocity=1000 -> lower=0 upper=+3.1416 effort=100 velocity=20
- joint motor_back_rightR_joint: limit lower=0 upper=+4.7124 effort=100 velocity=1000 -> lower=0 upper=+3.1416 effort=100 velocity=20
- joint motor_front_leftL_joint: limit lower=0 upper=+4.7124 effort=100 velocity=1000 -> lower=0 upper=+3.1416 effort=100 velocity=20
- joint motor_front_leftR_joint: limit lower=0 upper=+4.7124 effort=100 velocity=1000 -> lower=0 upper=+3.1416 effort=100 velocity=20
- joint motor_front_rightL_joint: limit lower=0 upper=+4.7124 effort=100 velocity=1000 -> lower=0 upper=+3.1416 effort=100 velocity=20
- joint motor_front_rightR_joint: limit lower=0 upper=+4.7124 effort=100 velocity=1000 -> lower=0 upper=+3.1416 effort=100 velocity=20
