Commit message: Perfect knee tracking with active thigh and ankle motion

File: frost-dev-master/example/minitaur/urdf/minitaur.urdf (robot description, URDF)
Before this commit: robot minitaur, 17 links, 16 joints
Joints:
- joint knee_back_leftL_link: limit effort=100 velocity=1000 -> lower=-3.14 upper=+3.14 effort=100 velocity=1000
- joint knee_back_leftR_link: limit effort=100 velocity=1000 -> lower=-3.14 upper=+3.14 effort=100 velocity=1000
- joint knee_back_rightL_link: limit effort=100 velocity=1000 -> lower=-3.14 upper=+3.14 effort=100 velocity=1000
- joint knee_front_leftL_link: limit effort=100 velocity=1000 -> lower=-3.14 upper=+3.14 effort=100 velocity=1000
- joint knee_front_leftR_link: limit effort=100 velocity=1000 -> lower=-3.14 upper=+3.14 effort=100 velocity=1000
- joint knee_front_rightL_link: limit effort=100 velocity=1000 -> lower=-3.14 upper=+3.14 effort=100 velocity=1000
- joint knee_front_rightR_link: limit effort=100 velocity=1000 -> lower=-3.14 upper=+3.14 effort=100 velocity=1000
- joint motor_back_leftL_joint: limit effort=100 velocity=1000 -> lower=-3.14 upper=+3.14 effort=100 velocity=1000
- joint motor_back_leftR_joint: limit effort=100 velocity=1000 -> lower=-3.14 upper=+3.14 effort=100 velocity=1000
- joint motor_back_rightL_joint: limit effort=100 velocity=1000 -> lower=-3.14 upper=+3.14 effort=100 velocity=1000
- joint motor_back_rightR_joint: limit effort=100 velocity=1000 -> lower=-3.14 upper=+3.14 effort=100 velocity=1000
- joint motor_front_leftL_joint: limit effort=100 velocity=1000 -> lower=-3.14 upper=+3.14 effort=100 velocity=1000
- joint motor_front_leftR_joint: limit effort=100 velocity=1000 -> lower=-3.14 upper=+3.14 effort=100 velocity=1000
- joint motor_front_rightL_joint: limit effort=100 velocity=1000 -> lower=-3.14 upper=+3.14 effort=100 velocity=1000
- joint motor_front_rightR_joint: limit effort=100 velocity=1000 -> lower=-3.14 upper=+3.14 effort=100 velocity=1000

Commit message: Debug URDF

File: frost-dev-master/example/minitaur/urdf/minitaur.urdf (robot description, URDF)
Before this commit: robot minitaur, 17 links, 16 joints
Joints:
- joint knee_back_rightR_link: limit effort=100 velocity=1000 -> lower=-3.14 upper=+3.14 effort=100 velocity=1000
